File: unid04_kicad/norgate/norgate.kicad_sch (KiCad schematic)
At the start: 11 parts, among them J1 Screw_Terminal_01x01, J2 Screw_Terminal_01x01, J3 Screw_Terminal_01x01, J4 Screw_Terminal_01x01, J5 Screw_Terminal_01x01, Q1 PMOS, Q2 PMOS, Q3 NMOS, Q4 NMOS, Q5 NMOS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

Commit message: Kicad nor gate project
Parts:
- removed Q1, Q2: PMOS, symbol Simulation_SPICE:PMOS
- removed Q3, Q4, Q5: NMOS, symbol Simulation_SPICE:NMOS
- removed Q6: PMOS, eteste, symbol Simulation_SPICE:PMOS
- added Q1, Q2, Q5: RE1C001ZPTL, PCM_SparkFun-Semiconductor-Standard:SC-89 SOT-490, symbol PCM_SparkFun-DiscreteSemi:Q_PMOS_0.1A_20V
- added Q3, Q4, Q7: RE1C002UNTCL, PCM_SparkFun-Semiconductor-Standard:SC-89 SOT-490, symbol PCM_SparkFun-DiscreteSemi:Q_NMOS_0.2A_20V
Connections:
- net GND: now also Q3.2 (S), Q4.2 (S), Q7.2 (S)
- net at J5.1 (Pin_1): now also Q2.3 (D), Q3.3 (D), Q4.3 (D), Q7.3 (D)
- net at J4.1 (Pin_1): now also Q2.1 (G), Q3.1 (G)
- net at J2.1 (Pin_1): now also Q4.1 (G), Q5.1 (G)
- net at J3.1 (Pin_1): now also Q1.1 (G), Q7.1 (G)
- net at J1.1 (Pin_1): now also Q5.2 (S)
- new net: Q1.3 (D), Q2.2 (S)
- new net: Q1.2 (S), Q5.3 (D)
